Commit message: need to change statemachine duration

File: robot_description/Ground/safe_climbing_test_2022/ground_3d_inclined.urdf (robot description, URDF)
Before this commit: robot ground_skeleton, 4 links, 3 joints
Links:
- link ground_link: geometry collision box size=1.0 1.0 5.00; visual box size=1.00 1.00 5.00
Joints:
- joint ground_flat_joint: origin xyz=0.0 0.0 -2.5 rpy=0 0.0 0.0 -> xyz=0.0 0.0 -2.0 rpy=0 0.0 0.0
- joint ground_joint: origin xyz=-0.7 0.0 0.0 rpy=0.6154796 -0.5235987 -0.9553166 -> xyz=0.0 0.0 0.0 rpy=0.6154796 -0.5235987 -0.9553166
