Commit message: office update

File: robot_description/Ground/safe_climbing_test_2022/hexa_column.urdf (robot description, URDF)
Before this commit: robot ground_skeleton, 4 links, 3 joints
Links:
- removed link wall_link
- added link ground, mass 1.0; collision box size=10 10 0.1; visual box size=10 10 0.1
- link ground_link: geometry collision mesh filename=meshes/hexa_column3.obj; visual mesh filename=meshes/hexa_column3.obj
Joints:
- removed joint wall_joint
- added joint ground_flat_joint: type fixed, parent world, child ground, origin xyz=0.0 0.0 0.0 rpy=0 0.0 0.0
- joint ground_joint: origin xyz=0 0 -0.01 rpy=0 1 0 -> xyz=-0.33 0.0 0.0 rpy=0. 0. 0.
