Commit message: hexa & slope test

File: robot_description/Ground/safe_climbing_test_2022/ground_inclined.urdf (robot description, URDF)
Before this commit: robot ground_skeleton, 4 links, 3 joints
Links:
- removed link ground
- added link wall_link; collision box size=50.0 50.0 2.3; visual box size=2.5 2.0 0.1
- link ground_link: geometry collision box size=5000.0 500.0 0.05; visual mesh filename=../mesh/tile_marble_diamond.dae scale=0.1 0.05 0.1
Joints:
- removed joint ground_flat_joint
- added joint wall_joint: type fixed, parent world, child wall_link, origin xyz=0.5 -0.1 -0.5 rpy=0 -0 0
- joint ground_joint: origin xyz=-0.33 0.0 0.0 rpy=0. 0. 0. -> xyz=0 0.5 -0.01 rpy=0 1 0

File: robot_description/Ground/safe_climbing_test_2022/slope.urdf (robot description, URDF)
Before this commit: robot ground_skeleton, 4 links, 3 joints
Links:
- link ground_link: geometry collision mesh filename=meshes/slope.obj; visual mesh filename=meshes/slope.obj
Joints:
- joint ground_flat_joint: origin xyz=0.0 0.0 0.0 rpy=0 0.0 0.0 -> xyz=0.0 0.0 -0.0 rpy=0 0.0 0.0
- joint ground_joint: origin xyz=-0.33 0.0 0.0 rpy=0. 0. 0. -> xyz=-0.05 -0.5 0.0 rpy=0. 1. 0.
