Commit message: first commit for anymal

File: robot_description/Robot/testobj/box.urdf (robot description, URDF)
Before this commit: robot 10kgbox, 8 links, 7 joints
Links:
- removed link base_link
- added link base, mass 10; collision box size=0.2 0.2 0.1; visual box size=0.2 0.2 0.1
Joints:
- joint baseRotX: child base_link -> base
- joint boxCOMtoCOP: parent base_link -> base
