Commit message: change the structure : fsm handle each task

File: robot_description/Robot/ANYmal/anymal_ur3.urdf (robot description, URDF)
Before this commit: robot anymalc-ur3, 92 links, 91 joints
Links:
- link ur3_base: mass 2.000 -> 1.000
- link ur3_ee_link: mass 5.000 -> 0.100
- link ur3_forearm_link: mass 1.260 -> 1.000
- link ur3_shoulder_link: mass 2.000 -> 1.000
- link ur3_upper_arm_link: mass 3.420 -> 1.000
